File: Electrical/PCB Projects/64 Bit - Main Board/Connectors.kicad_sch (KiCad schematic)
At the start: 33 parts, among them J1 61301021821, J14 1985195, J15 Conn_01x09, J16 Conn_01x09, J2 61301021821, J3 61301021821, J4 M20-7920242R, J5 USBC, J7 PJ-102A, P1 Conn_01x02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

Commit message: finalized schematic, made ESP32 footprint, started PCB update
Parts:
- added D47: SK54BLF-R1_00001, Footprint drive Dump 1:SK54BLF-R1_00001, symbol HDD_CLK_V6.0:SK54BLF-R1_00001
- U9: footprint (none) -> Footprint drive Dump 1:ESP32-C6-LCD-1.47
Connections:
- net at U9.1 (5V): now also D47.1 (K); no longer JP1.1 (A)
- new net: D47.2 (A), JP1.1 (A)
Other:
- moved on the sheet: JP1

Commit message: small pcb layout work
Connections:
- net +5V: now also D47.2 (A); no longer JP1.2 (B)
- net at U9.1 (5V): now also JP1.1 (A); no longer D47.1 (K)
- new net: D47.1 (K), JP1.2 (B)
Other:
- moved on the sheet: D47, JP1
Changed lines of the file:
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@@
 	(wire
 		(pts
-			(xy 238.76 86.36) (xy 238.76 90.17)
+			(xy 213.36 49.53) (xy 215.9 49.53)
 		)
 		(stroke
@@
 	(wire
 		(pts
-			(xy 213.36 49.53) (xy 215.9 49.53)
+			(xy 237.49 39.37) (xy 237.49 43.18)
 		)
 		(stroke
@@
 	(wire
 		(pts
-			(xy 237.49 39.37) (xy 237.49 43.18)
+			(xy 210.82 156.21) (xy 210.82 162.56)
 		)
 		(stroke
@@
 	(wire
 		(pts
-			(xy 210.82 156.21) (xy 210.82 162.56)
+			(xy 243.84 88.9) (xy 238.76 88.9)
 		)
 		(stroke
@@
 	(wire
 		(pts
-			(xy 254 86.36) (xy 257.81 86.36)
-		)
-		(stroke
-			(width 0)
-			(type default)
-		)
-	)
-	(wire
-		(pts
 			(xy 36.83 130.81) (xy 36.83 128.27)
 		)
@@
 	(wire
 		(pts
-			(xy 243.84 86.36) (xy 238.76 86.36)
-		)
-		(stroke
-			(width 0)
-			(type default)
-		)
-	)
-	(wire
-		(pts
 			(xy 109.22 38.1) (xy 123.19 38.1)
 		)
@@
 		)
 	)
+	(wire
+		(pts
+			(xy 257.81 85.09) (xy 257.81 88.9)
+		)
+		(stroke
+			(width 0)
+			(type default)
+		)
+	)
 	(polyline
 		(pts
@@
 	(wire
 		(pts
-			(xy 198.12 49.53) (xy 200.66 49.53)
+			(xy 238.76 100.33) (xy 238.76 102.87)
 		)
 		(stroke
@@
 	(wire
 		(pts
-			(xy 160.02 110.49) (xy 160.02 113.03)
+			(xy 198.12 49.53) (xy 200.66 49.53)
 		)
 		(stroke
@@
 	(wire
 		(pts
-			(xy 213.36 44.45) (xy 220.98 44.45)
+			(xy 160.02 110.49) (xy 160.02 113.03)
 		)
 		(stroke
@@
 	(wire
 		(pts
-			(xy 237.49 58.42) (xy 264.16 58.42)
+			(xy 213.36 44.45) (xy 220.98 44.45)
 		)
 		(stroke
@@
 	(wire
 		(pts
-			(xy 238.76 97.79) (xy 238.76 102.87)
+			(xy 237.49 58.42) (xy 264.16 58.42)
 		)
 		(stroke
@@
 	(wire
 		(pts
+			(xy 251.46 88.9) (xy 257.81 88.9)
+		)
+		(stroke
+			(width 0)
+			(type default)
+		)
+	)
+	(wire
+		(pts
 			(xy 276.86 118.11) (xy 276.86 129.54)
 		)
@@
 	(wire
 		(pts
+			(xy 238.76 88.9) (xy 238.76 90.17)
+		)
+		(stroke
+			(width 0)
+			(type default)
+		)
+	)
+	(wire
+		(pts
 			(xy 267.97 107.95) (xy 274.32 107.95)
 		)
@@
 	(wire
 		(pts
-			(xy 257.81 86.36) (xy 257.81 83.82)
-		)
-		(stroke
-			(width 0)
-			(type default)
-		)
-	)
-	(wire
-		(pts
 			(xy 236.22 110.49) (xy 236.22 102.87)
 		)
@@
 	(symbol
 		(lib_id "HDD_CLK_V6.0:SK54BLF-R1_00001")
-		(at 238.76 93.98 90)
+		(at 247.65 88.9 0)
 		(unit 1)
 		(exclude_from_sim no)
@@
 		(dnp no)
 		(property "Reference" "D47"
-			(at 241.3 95.25 0)
+			(at 246.38 91.44 0)
 			(effects
 				(font
@@
 		)
 		(property "Value" "SK54BLF-R1_00001"
-			(at 234.95 100.33 0)
+			(at 235.204 85.344 0)
 			(effects
 				(font
@@
 		)
 		(property "Footprint" "Footprint drive Dump 1:SK54BLF-R1_00001"
-			(at 238.76 93.98 0)
+			(at 247.65 88.9 0)
 			(effects
 				(font
@@
 		)
 		(property "Datasheet" "~"
-			(at 238.76 93.98 0)
+			(at 247.65 88.9 0)
 			(effects
 				(font
@@
 		)
 		(property "Description" ""
-			(at 238.76 93.98 0)
+			(at 247.65 88.9 0)
 			(effects
 				(font
@@
 	(symbol
 		(lib_id "power:+5V")
-		(at 257.81 83.82 0)
+		(at 257.81 85.09 0)
 		(unit 1)
 		(exclude_from_sim no)
@@
 		(on_board yes)
 		(dnp no)
-		(fields_autoplaced yes)
 		(property "Reference" "#PWR0128"
-			(at 257.81 87.63 0)
+			(at 257.81 88.9 0)
 			(effects
 				(font
@@
 		)
 		(property "Value" "+5V"
-			(at 260.35 82.5499 0)
+			(at 256.032 80.772 0)
 			(effects
 				(font
@@
 		)
 		(property "Footprint" ""
-			(at 257.81 83.82 0)
+			(at 257.81 85.09 0)
 			(effects
 				(font
@@
 		)
 		(property "Datasheet" ""
-			(at 257.81 83.82 0)
+			(at 257.81 85.09 0)
 			(effects
 				(font
@@
 		)
 		(property "Description" "Power symbol creates a global label with name \"+5V\""
-			(at 257.81 83.82 0)
+			(at 257.81 85.09 0)
 			(effects
 				(font
@@
 	(symbol
 		(lib_id "Jumper:Jumper_2_Open")
-		(at 248.92 86.36 0)
+		(at 238.76 95.25 90)
 		(unit 1)
 		(exclude_from_sim no)
@@
 		(dnp no)
 		(property "Reference" "JP1"
-			(at 250.444 88.646 0)
+			(at 241.046 93.726 0)
 			(effects
 				(font
@@
 		)
 		(property "Value" "Jumper_2_Open"
-			(at 256.286 83.058 0)
+			(at 235.458 87.884 0)
 			(effects
 				(font
@@
 		)
 		(property "Footprint" "Connector_PinHeader_2.54mm:PinHeader_1x02_P2.54mm_Vertical"
-			(at 248.92 86.36 0)
+			(at 238.76 95.25 0)
 			(effects
 				(font
@@
 		)
 		(property "Datasheet" "~"
-			(at 248.92 86.36 0)
+			(at 238.76 95.25 0)
 			(effects
 				(font
@@
 		)
 		(property "Description" "Jumper, 2-pole, open"
-			(at 248.92 86.36 0)
+			(at 238.76 95.25 0)
 			(effects
 				(font
