File: Electrical/PCB Projects/64 Bit - Main Board/Level Shifting.kicad_sch (KiCad schematic)
At the start: 42 parts, among them U4 74HC3G34DC, U5 74HC3G34DC, U6 74HC3G34DC

Commit message: slight changes
Changed lines of the file:
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@@
 		)
 		(property "Value" "0.1uF_0603"
-			(at 127 78.74 90)
+			(at 126.492 79.756 90)
 			(effects
 				(font
