File: Electrical/PCB Projects/64 Bit - Main Board/Power.kicad_sch (KiCad schematic)
At the start: 34 parts, among them K4 PR30-5V-450-1A-E, K5 PR30-12V-450-1A-E, Q10 XP231P0201TR-G, SW5 L102011MS02Q, SW6 power_switch

Commit message: adding comments after build. Documentation for next revision
Other:
- note added: "P-Channel not suitable try: SQ2389CES-T1_GE3 default gate voltage must be 12V"
- note added: "power switch doesnt have enough room"
Changed lines of the file:
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@@
+		)
+	)
+	(text "P-Channel not suitable try: \nSQ2389CES-T1_GE3\ndefault gate voltage must be 12V"
+		(exclude_from_sim no)
+		(at 120.904 105.41 0)
+		(effects
+			(font
+				(size 1.905 1.905)
+				(thickness 0.381)
+				(bold yes)
+				(color 255 46 77 1)
+			)
+			(justify left)
 		)
 	)
@@
 			)
 			(justify left)
+		)
+	)
+	(text "power switch doesnt\nhave enough room"
+		(exclude_from_sim no)
+		(at 50.292 35.56 0)
+		(effects
+			(font
+				(size 1.905 1.905)
+				(thickness 0.381)
+				(bold yes)
+				(color 255 46 77 1)
+			)
+			(justify left)
