File: Electrical/PCB Projects/64 Bit - LED Board/64 Bit - LED Board.kicad_sch (KiCad schematic)
At the start: 15 parts, among them P1 Conn_01x03, P2 Conn_01x03

Commit message: near final state. Includes BOM, price, etc
Other:
- company: (none) -> Kadin Whiting
- title: (none) -> 64 Bit - LED Board
Changed lines of the file:
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@@
 	(generator_version "9.0")
 	(paper "A4")
+	(title_block
+		(title "64 Bit - LED Board")
+		(date "2025-12-01")
+		(rev "1")
+		(company "Kadin Whiting")
+	)
 	(rectangle
 		(start 31.75 69.088)
