File: Electrical/PCB Projects/64 Bit - LED Board/64 Bit - LED Board.kicad_pcb (KiCad board)
At the start: 2 copper layers, 160.1 x 30 mm, 17 parts, among them P1 Conn_01x03, P2 Conn_01x03

Commit message: near final state. Includes BOM, price, etc
Other:
- board text added: "'64 Bit' Nixie Tube Clock - LED Board_V1.0 Dec 2025"
- board text removed: "'64 Bit' Nixie Tube Clock - LED Board_V1.0 Oct 2025"
Changed lines of the file:
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@@
 			(drillshape 0)
 			(scaleselection 1)
-			(outputdirectory "G:/My Drive/Projects (GDrive)/31_My First Nixie Clock/01_My First Nixie Clock/PCB Plots/LED Board/Gerber Files/")
+			(outputdirectory "C:/Users/Kadin/Desktop/Git Projects/64-Bit/Electrical/PCB Outputs/64 Bit - LED Board/gerbers/")
 		)
 	)
@@
 		(layer "User.2")
 	)
-	(gr_text "'64 Bit' Nixie Tube Clock - LED Board_V1.0 Oct 2025"
+	(gr_text "'64 Bit' Nixie Tube Clock - LED Board_V1.0 Dec 2025"
 		(at 80.1 114.3 0)
 		(layer "F.Mask")
@@
 		)
 	)
-	(gr_text "'64 Bit' Nixie Tube Clock - LED Board_V1.0 Oct 2025"
-		(at 121.298712 114.239638 -0)
+	(gr_text "'64 Bit' Nixie Tube Clock - LED Board_V1.0 Dec 2025"
+		(at 121.298712 114.239638 0)
 		(layer "B.Mask")
 		(effects
